File: Peripherical Mimetizer/mimetizer.sch (KiCad schematic (older format))
At the start: 29 parts, among them J1 TC2030, U1 Nrf52810-QCAA, U2 BME280, Y1 32,768KHz, Y2 32MHz

Commit message: Schematics Done
Parts:
- removed U2: BME280, Package_LGA:Bosch_LGA-8_2.5x2.5mm_P0.65mm_ClockwisePinNumbering, symbol Sensor:BME280
- added C15: 22pF, Capacitor_SMD:C_0402_1005Metric, symbol Device:C_Small
- added C16: 10nF, Capacitor_SMD:C_0402_1005Metric, symbol Device:C_Small
- added J2: USB_B_Mini, symbol Connector:USB_B_Mini
- added R4: 22, Resistor_SMD:R_0402_1005Metric, symbol Device:R_Small_US
- added R5, R6: 10k, Resistor_SMD:R_0402_1005Metric, symbol Device:R_Small_US
- added SW1: SW_Push, symbol Switch:SW_Push
- added U2: ATmega32U4-AU, Package_QFP:TQFP-44_10x10mm_P0.8mm, symbol MCU_Microchip_ATmega:ATmega32U4-AU
- added Y3: Crystal_GND2, symbol Device:Crystal_GND2
- C13: value 100nF -> 22pF
- C14: value 100nF -> 1uF
- R3: value 1k -> 22
Connections:
- net GND: now also C13.1, C14.1, C15.1, C16.2, J2.5 (GND), J2.6 (Shield), R6.2, SW1.1, U2.15 (GND), U2.23 (GND), U2.35 (GND), U2.43 (GND), U2.5 (UGND), Y3.2; no longer C13.2, C14.2, R3.2
- net SWCLK: no longer U1.17 (SWDCLK)
- net SWDIO: no longer U1.18 (SWDIO)
- net VDD: now also C16.1, J2.1 (VBUS), R5.1, U2.14 (VCC), U2.2 (UVCC), U2.24 (AVCC), U2.34 (VCC), U2.44 (AVCC), U2.7 (VBUS); no longer C13.1, C14.1
- net PB0: now reaches U1.10 (P0.12)
- net PB1: now reaches U1.11 (P0.14)
- net PB2: now reaches U1.12 (P0.15)
- net PB3: now reaches U1.13 (P0.16)
- net at R3.1: now also J2.3 (D+)
- net ANT: no longer names the net of U1.19 (ANT)
- net SCL: no longer names the net of R2.2, U1.7 (P0.09)
- net SDA: no longer names the net of R1.2, U1.8 (P0.10)
- new net: R5.2, SW1.2, U2.13 (~RESET)
- new net: C15.2, U2.16 (XTAL2), Y3.1
- new net: R4.2, U2.3 (D-)
- new net: R6.1, U2.33 (~HWB~/PE2)
- new net: R3.2, U2.4 (D+)
- new net: C14.2, U2.6 (UCAP)
- new net: J2.2 (D-), R4.1
- new net: C13.2, Y3.3
- new net P0.12: U2.8 (PB0)
- new net P0.14: U2.9 (PB1)
- new net P0.15: U2.10 (PB2)
- new net P0.16: U2.11 (PB3)
- no-connect marks 14 -> 36
Other:
- note added: "MCU 1 - NRF52810"
- note added: "MCU 2 - ATMEGA32U4\n"
- note removed: "MCU - NRF52810"
- note removed: "SENSOR - BME280"
- moved on the sheet: BT1, C1, C10, C11, C12, C2, C3, C4, C5, C6, C7, C8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
