File: RX23W/RX23W.sch (KiCad schematic (older format))
At the start: 32 parts, among them J1 USB_B_Micro, J2 TC2030, SW1 SW_Push, U1 LMR10515, U2 USBLC6-2SC6, U3 RX23W, Y1 54MHz

Commit message: Commit Inicial de Janeiro
Connections:
- net VDD: no longer C10.1, C5.1, C9.1, D3.2 (A), L1.2, R4.1, U3.34 (VCC), U3.36 (VSS), U3.9 (VCC)
- new net VCC: C10.1, C5.1, C9.1, D3.2 (A), L1.2, R4.1, U3.34 (VCC), U3.36 (VSS), U3.9 (VCC)
Changed lines of the file:
@@
-$EndComp
-$Comp
-L power:VDD #PWR019
-U 1 1 5DFFA7AD
-P 8950 5150
-F 0 "#PWR019" H 8950 5000 50  0001 C CNN
-F 1 "VDD" H 8967 5323 50  0000 C CNN
-F 2 "" H 8950 5150 50  0001 C CNN
-F 3 "" H 8950 5150 50  0001 C CNN
-	1    8950 5150
-	1    0    0    -1
 $EndComp
 $Comp
@@
 	1    0    0    -1
 $EndComp
-$Comp
-L power:VDD #PWR017
-U 1 1 5DFFEB25
-P 8450 1950
-F 0 "#PWR017" H 8450 1800 50  0001 C CNN
-F 1 "VDD" H 8467 2123 50  0000 C CNN
-F 2 "" H 8450 1950 50  0001 C CNN
-F 3 "" H 8450 1950 50  0001 C CNN
-	1    8450 1950
-	1    0    0    -1
-$EndComp
 Wire Wire Line
 	8450 2150 8450 2050
 Wire Wire Line
 	8800 2850 8800 2600
-Connection ~ 8450 2050
-Wire Wire Line
-	8450 2050 8450 1950
 Wire Wire Line
 	8000 5450 8600 5450
@@
 Wire Wire Line
 	2350 3400 2350 3750
-$Comp
-L power:VDD #PWR012
-U 1 1 5E0BA8D1
-P 3900 3300
-F 0 "#PWR012" H 3900 3150 50  0001 C CNN
-F 1 "VDD" H 3917 3473 50  0000 C CNN
-F 2 "" H 3900 3300 50  0001 C CNN
-F 3 "" H 3900 3300 50  0001 C CNN
-	1    3900 3300
-	1    0    0    -1
-$EndComp
 Wire Wire Line
 	3900 3400 3900 3650
-Wire Wire Line
-	3900 3300 3900 3400
 Connection ~ 3900 3400
 Wire Wire Line
@@
 Wire Wire Line
 	8800 5250 8950 5250
-Connection ~ 8950 5250
-Wire Wire Line
-	8950 5250 8950 5400
-Wire Wire Line
-	8950 5150 8950 5250
 Wire Wire Line
 	9700 5250 9300 5250
@@
 $EndComp
 NoConn ~ 9200 4850
+Text Label 3950 3250 0    50   ~ 0
+3.3V
+Text Label 850  2800 0    50   ~ 0
+5V
+Text Label 2900 6650 0    50   ~ 0
+5V
+$Comp
+L power:VDD #PWR?
+U 1 1 5DFE7677
+P 2250 5200
+F 0 "#PWR?" H 2250 5050 50  0001 C CNN
+F 1 "VDD" H 2267 5373 50  0000 C CNN
+F 2 "" H 2250 5200 50  0001 C CNN
+F 3 "" H 2250 5200 50  0001 C CNN
+	1    2250 5200
+	1    0    0    -1
+$EndComp
+Text Label 2300 5150 0    50   ~ 0
+5V
+Text Label 4600 4300 0    50   ~ 0
+OLHAESSERESISTORAQUI
+Text Label 9800 5700 0    50   ~ 0
+OLHAESSERESISTORAQUI
+Text Label 3500 7400 0    50   ~ 0
+OLHAESSERESISTORAQUI
+$Comp
+L power:VCC #PWR?
+U 1 1 5DFF57AC
+P 3900 3300
+F 0 "#PWR?" H 3900 3150 50  0001 C CNN
+F 1 "VCC" H 3917 3473 50  0000 C CNN
+F 2 "" H 3900 3300 50  0001 C CNN
+F 3 "" H 3900 3300 50  0001 C CNN
+	1    3900 3300
+	1    0    0    -1
+$EndComp
+Wire Wire Line
+	3900 3300 3900 3400
+Text Label 8500 1950 0    50   ~ 0
+3.3V
+$Comp
+L power:VCC #PWR?
+U 1 1 5E002F62
+P 8450 2000
+F 0 "#PWR?" H 8450 1850 50  0001 C CNN
+F 1 "VCC" H 8467 2173 50  0000 C CNN
+F 2 "" H 8450 2000 50  0001 C CNN
+F 3 "" H 8450 2000 50  0001 C CNN
+	1    8450 2000
+	1    0    0    -1
+$EndComp
+Wire Wire Line
+	8450 2000 8450 2050
+Connection ~ 8450 2050
+Text Label 9000 5100 0    50   ~ 0
+3.3V
+$Comp
+L power:VCC #PWR?
+U 1 1 5E0108A9
+P 8950 5150
+F 0 "#PWR?" H 8950 5000 50  0001 C CNN
+F 1 "VCC" H 8967 5323 50  0000 C CNN
+F 2 "" H 8950 5150 50  0001 C CNN
+F 3 "" H 8950 5150 50  0001 C CNN
+	1    8950 5150
+	1    0    0    -1
+$EndComp
+Wire Wire Line
+	8950 5150 8950 5250
+Connection ~ 8950 5250
+Wire Wire Line
+	8950 5250 8950 5400
+Text Label 3950 700  0    50   ~ 0
+OLHARISSOAQUISETEMRESET
+Text Label 1800 2700 0    50   ~ 0
+ARRUMAISSOAQUI
 $EndSCHEMATC
